Commit message: move laser arm above

File: robot_description_rm20/urdf/robot_description_rm20_mid360.xacro (robot description, xacro)
@@ -114,6 +114,8 @@
   </link>
   <joint name="laser_static" type="fixed">
-    <origin xyz="0.144 0 0.2475" rpy="0 0 0" />
-    <parent link="base_link" />
+    <!-- <origin xyz="0.144 0 0.2475" rpy="0 0 0" /> -->
+    <origin xyz="0 0 0.4" rpy="0 0 0" />
+    <!-- <parent link="base_link" /> -->
+    <parent link="arm" />
     <child link="laser" />
     <axis xyz="0 0 0" />
